Commit message: working old version

File: mycobot_description/urdf/mycobot_urdf.urdf.xacro (robot description, xacro)
@@ -2,105 +2,105 @@
 <robot  xmlns:xacro="http://www.ros.org/wiki/xacro" name="firefighter" >
 <xacro:property name="width" value=".2" />
-  <link name="joint1">
+  <link name="base_link">
     <visual>
       <geometry>
 	     <!--- 0.0 0 -0.04  1.5708 3.14159-->
-       <mesh filename="package://mycobot_description/urdf/280jn/joint1_jet.dae"/>
+       <mesh filename="package://mycobot_description/urdf/joint1_jet.dae"/>
       </geometry>
     <origin xyz = "0.0 0 0 " rpy = " 0 0 3.14159"/>
     </visual>
   </link>
-  <link name="joint2">
+  <link name="link_joint2">
     <visual>
       <geometry>
-       <mesh filename="package://mycobot_description/urdf/280jn/joint2.dae"/>
+       <mesh filename="package://mycobot_description/urdf/joint2.dae"/>
       </geometry>
     <origin xyz = "0.0 0 -0.06096 " rpy = " 0 0 -1.5708"/>
     </visual>
   </link>
-  <link name="joint3">
+  <link name="link_joint3">
     <visual>
       <geometry>
-       <mesh filename="package://mycobot_description/urdf/280jn/joint3.dae"/>
+       <mesh filename="package://mycobot_description/urdf/joint3.dae"/>
       </geometry>
     <origin xyz = "0.0 0 0.03256 " rpy = " 0 -1.5708 0"/>
     </visual>
   </link>
-  <link name="joint4">
+  <link name="link_joint4">
     <visual>
       <geometry>
        <!--- 0.0 0 -0.04 -->
-       <mesh filename="package://mycobot_description/urdf/280jn/joint4.dae"/>
+       <mesh filename="package://mycobot_description/urdf/joint4.dae"/>
       </geometry>
     <origin xyz = "0.0 0 0.03056 " rpy = " 0 -1.5708 0"/>
     </visual>
   </link>
-<link name="joint5">
+<link name="link_joint5">
     <visual>
       <geometry>
        <!--- 0.0 0 -0.04 -->
-       <mesh filename="package://mycobot_description/urdf/280jn/joint5.dae"/>
+       <mesh filename="package://mycobot_description/urdf/joint5.dae"/>
       </geometry>
     <origin xyz = "0.0 0 -0.03356 " rpy = " 0 -1.5708 1.5708"/>
     </visual>
   </link>
-  <link name="joint6">
+  <link name="link_joint6">
     <visual>
       <geometry>
        <!--- 0.0 0 -0.04 -->
-       <mesh filename="package://mycobot_description/urdf/280jn/joint6.dae"/>
+       <mesh filename="package://mycobot_description/urdf/joint6.dae"/>
       </geometry>
     <origin xyz = "0 0.00 -0.038 " rpy = " 0 0 0"/>
     </visual>
   </link>
-  <link name="joint6_flange">
+  <link name="link_joint6_flange">
     <visual>
       <geometry>
        <!--- 0.0 0 -0.04 -->
-       <mesh filename="package://mycobot_description/urdf/280jn/joint7.dae"/>
+       <mesh filename="package://mycobot_description/urdf/joint7.dae"/>
       </geometry>
     <origin xyz = "0.0 0 -0.012 " rpy = " 0 0 0"/>
     </visual>
   </link>
-    <joint name="joint2_to_joint1" type="revolute">
+    <joint name="joint_1" type="revolute">
     <axis xyz="0 0 1"/>
     <limit effort = "1000.0" lower = "-3.14" upper = "3.14159" velocity = "0"/>
-    <parent link="joint1"/>
-    <child link="joint2"/>
+    <parent link="base_link"/>
+    <child link="link_joint2"/>
     <origin xyz= "0 0 0.15756" rpy = "0 0 0"/>
   </joint>
-  <joint name="joint3_to_joint2" type="revolute">
+  <joint name="joint_2" type="revolute">
     <axis xyz="0 0 1"/>
     <limit effort = "1000.0" lower = "-3.14" upper = "3.14159" velocity = "0"/>
-    <parent link="joint2"/>
-    <child link="joint3"/>
+    <parent link="link_joint2"/>
+    <child link="link_joint3"/>
     <origin xyz= "0 0 -0.001" rpy = "0 1.5708 -1.5708"/>
   </joint>
-  <joint name="joint4_to_joint3" type="revolute">
+  <joint name="joint_3" type="revolute">
     <axis xyz=" 0 0 1"/>
     <limit effort = "1000.0" lower = "-3.14" upper = "3.14159" velocity = "0"/>
-    <parent link="joint3"/>
-    <child link="joint4"/>
+    <parent link="link_joint3"/>
+    <child link="link_joint4"/>
     <origin xyz= "  -0.1104 0 0   " rpy = "0 0 0"/>
   </joint>
-  <joint name="joint5_to_joint4" type="revolute">
+  <joint name="joint_4" type="revolute">
     <axis xyz=" 0 0 1"/>
     <limit effort = "1000.0" lower = "-3.14" upper = "3.14159" velocity = "0"/>
-    <parent link="joint4"/>
-    <child link="joint5"/>
+    <parent link="link_joint4"/>
+    <child link="link_joint5"/>
     <origin xyz= "-0.096 0 0.06462" rpy = "0 0 -1.5708"/>
   </joint>
-  <joint name="joint6_to_joint5" type="revolute">
+  <joint name="joint_5" type="revolute">
     <axis xyz="0 0 1"/>
     <limit effort = "1000.0" lower = "-3.14" upper = "3.14159" velocity = "0"/>
-    <parent link="joint5"/>
-    <child link="joint6"/>
+    <parent link="link_joint5"/>
+    <child link="link_joint6"/>
     <origin xyz= "0 -0.07318 0" rpy = "1.5708 -1.5708 0"/>
   </joint>
-  <joint name="joint6output_to_joint6" type="revolute">
+  <joint name="joint_6" type="revolute">
     <axis xyz="0 0 1"/>
     <limit effort = "1000.0" lower = "-3.14" upper = "3.14159" velocity = "0"/>
-    <parent link="joint6"/>
-    <child link="joint6_flange"/>
+    <parent link="link_joint6"/>
+    <child link="link_joint6_flange"/>
     <origin xyz= "0 0.0456 0" rpy = "-1.5708 0 0"/>
   </joint>

Commit message: fix gazebo show

File: mycobot_description/urdf/mycobot_urdf.urdf.xacro (robot description, xacro)
@@ -1,6 +1,18 @@
 <?xml version="1.0"?>
-<robot  xmlns:xacro="http://www.ros.org/wiki/xacro" name="firefighter" >
-<xacro:property name="width" value=".2" />
+<robot  xmlns:xacro="http://www.ros.org/wiki/xacro" name="mycobot" >
+    <xacro:property name="width" value=".2" />
+    <!-- Useful Variables (Properties) -->
+    <xacro:property name="PI" value="3.14159265359" />
+    <xacro:property name="effort" value="30" />
+    <xacro:property name="velocity" value="10" />
+    <xacro:macro name="default_interial" params="mass">
+        <inertial>
+            <mass value="${mass}"/>
+            <inertia ixx="1" ixy="0.0" ixz="0.0" iyy="1" iyz="0.0" izz="1"/>
+        </inertial>
+    </xacro:macro>
+  <link name="world"/>
   <link name="base_link">
+  <xacro:default_interial mass="1.0"/>
     <visual>
       <geometry>
@@ -10,6 +22,14 @@
     <origin xyz = "0.0 0 0 " rpy = " 0 0 3.14159"/>
     </visual>
+    <collision>
+      <geometry>
+	     <!--- 0.0 0 -0.04  1.5708 3.14159-->
+       <mesh filename="package://mycobot_description/urdf/joint1_jet.dae"/>
+      </geometry>
+    <origin xyz = "0.0 0 0 " rpy = " 0 0 3.14159"/>
+    </collision>
   </link>
   <link name="link_joint2">
+  <xacro:default_interial mass="0.5"/>
     <visual>
       <geometry>
@@ -18,6 +38,13 @@
     <origin xyz = "0.0 0 -0.06096 " rpy = " 0 0 -1.5708"/>
     </visual>
+    <collision>
+      <geometry>
+       <mesh filename="package://mycobot_description/urdf/joint2.dae"/>
+      </geometry>
+    <origin xyz = "0.0 0 -0.06096 " rpy = " 0 0 -1.5708"/>
+    </collision>
   </link>
   <link name="link_joint3">
+  <xacro:default_interial mass="0.5"/>
     <visual>
       <geometry>
@@ -26,6 +53,13 @@
     <origin xyz = "0.0 0 0.03256 " rpy = " 0 -1.5708 0"/>
     </visual>
+    <collision>
+      <geometry>
+       <mesh filename="package://mycobot_description/urdf/joint3.dae"/>
+      </geometry>
+    <origin xyz = "0.0 0 0.03256 " rpy = " 0 -1.5708 0"/>
+    </collision>
   </link>
   <link name="link_joint4">
+  <xacro:default_interial mass="0.5"/>
     <visual>
       <geometry>
@@ -35,15 +69,29 @@
     <origin xyz = "0.0 0 0.03056 " rpy = " 0 -1.5708 0"/>
     </visual>
+    <collision>
+      <geometry>
+       <!--- 0.0 0 -0.04 -->
+       <mesh filename="package://mycobot_description/urdf/joint4.dae"/>
+      </geometry>
+    <origin xyz = "0.0 0 0.03056 " rpy = " 0 -1.5708 0"/>
+    </collision>
   </link>
 <link name="link_joint5">
+  <xacro:default_interial mass="0.4"/>
     <visual>
       <geometry>
-       <!--- 0.0 0 -0.04 -->
        <mesh filename="package://mycobot_description/urdf/joint5.dae"/>
       </geometry>
-    <origin xyz = "0.0 0 -0.03356 " rpy = " 0 -1.5708 1.5708"/>
+      <origin xyz = "0.0 0 -0.03356 " rpy = " 0 -1.5708 1.5708"/>
     </visual>
+    <collision>
+      <geometry>
+       <mesh filename="package://mycobot_description/urdf/joint5.dae"/>
+      </geometry>
+      <origin xyz = "0.0 0 -0.03356 " rpy = " 0 -1.5708 1.5708"/>
+    </collision>
   </link>
   <link name="link_joint6">
+  <xacro:default_interial mass="0.5"/>
     <visual>
       <geometry>
@@ -53,6 +101,14 @@
     <origin xyz = "0 0.00 -0.038 " rpy = " 0 0 0"/>
     </visual>
+    <collision>
+      <geometry>
+       <!--- 0.0 0 -0.04 -->
+       <mesh filename="package://mycobot_description/urdf/joint6.dae"/>
+      </geometry>
+    <origin xyz = "0 0.00 -0.038 " rpy = " 0 0 0"/>
+    </collision>
   </link>
   <link name="link_joint6_flange">
+  <xacro:default_interial mass="0.05"/>
     <visual>
       <geometry>
@@ -62,5 +118,18 @@
     <origin xyz = "0.0 0 -0.012 " rpy = " 0 0 0"/>
     </visual>
+    <collision>
+      <geometry>
+       <!--- 0.0 0 -0.04 -->
+       <mesh filename="package://mycobot_description/urdf/joint7.dae"/>
+      </geometry>
+    <origin xyz = "0.0 0 -0.012 " rpy = " 0 0 0"/>
+    </collision>
   </link>
+      <!-- Joints -->
+    <joint name="virtual_joint" type="fixed">
+        <parent link="world"/>
+        <child link="base_link"/>
+        <origin xyz="0 0 0" rpy="0 0 0"/>
+    </joint>
     <joint name="joint_1" type="revolute">
     <axis xyz="0 0 1"/>

Commit message: working gazebo model with controller

File: mycobot_description/urdf/mycobot_urdf.urdf.xacro (robot description, xacro)
@@ -78,16 +78,18 @@
   </link>
 <link name="link_joint5">
-  <xacro:default_interial mass="0.4"/>
-    <visual>
-      <geometry>
+  <xacro:default_interial mass="0.5"/>
+    <visual>
+      <geometry>
+       <!--- 0.0 0 -0.04 -->
        <mesh filename="package://mycobot_description/urdf/joint5.dae"/>
       </geometry>
-      <origin xyz = "0.0 0 -0.03356 " rpy = " 0 -1.5708 1.5708"/>
-    </visual>
-    <collision>
-      <geometry>
+    <origin xyz = "0.0 0 -0.03356 " rpy = " 0 -1.5708 1.5708"/>
+    </visual>
+    <collision>
+      <geometry>
+       <!--- 0.0 0 -0.04 -->
        <mesh filename="package://mycobot_description/urdf/joint5.dae"/>
       </geometry>
-      <origin xyz = "0.0 0 -0.03356 " rpy = " 0 -1.5708 1.5708"/>
+    <origin xyz = "0.0 0 -0.03356 " rpy = " 0 -1.5708 1.5708"/>
     </collision>
   </link>
@@ -174,3 +176,55 @@
     <origin xyz= "0 0.0456 0" rpy = "-1.5708 0 0"/>
   </joint>
+  <ros2_control name="GazeboSimSystem" type="system">
+  <hardware>
+    <plugin>gazebo_ros2_control/GazeboSystem</plugin>
+  </hardware>
+    <joint name="joint_1">
+        <command_interface name="position"/>
+        <state_interface name="position">
+            <param name="initial_value">0.0</param>
+        </state_interface>
+        <state_interface name="velocity"/>
+    </joint>
+    <joint name="joint_2">
+        <command_interface name="position"/>
+        <state_interface name="position">
+            <param name="initial_value">0.0</param>
+        </state_interface>
+        <state_interface name="velocity"/>
+    </joint>
+    <joint name="joint_3">
+        <command_interface name="position"/>
+        <state_interface name="position">
+            <param name="initial_value">0.0</param>
+        </state_interface>
+        <state_interface name="velocity"/>
+    </joint>
+    <joint name="joint_4">
+        <command_interface name="position"/>
+        <state_interface name="position">
+            <param name="initial_value">0.0</param>
+        </state_interface>
+        <state_interface name="velocity"/>
+    </joint>
+    <joint name="joint_5">
+        <command_interface name="position"/>
+        <state_interface name="position">
+            <param name="initial_value">0.0</param>
+        </state_interface>
+        <state_interface name="velocity"/>
+    </joint>
+    <joint name="joint_6">
+        <command_interface name="position"/>
+        <state_interface name="position">
+            <param name="initial_value">0.0</param>
+        </state_interface>
+        <state_interface name="velocity"/>
+    </joint>
+  </ros2_control>
+  <gazebo>
+    <plugin name="gazebo_ros2_control" filename="libgazebo_ros2_control.so">
+      <parameters>$(find mycobot_280)/config/mycobot_controllers.yaml</parameters>
+    </plugin>
+  </gazebo>
 </robot>
